Commit message: shell_scripts added

File: src/rsk_bot/urdf/common_properties.xacro (robot description, xacro)
@@ -1,7 +1,13 @@
-<?xml version="1.0"?>
-<robot>
-  <!-- Various materials' property which can be used in the robot -->
+<?xml version="1.0" ?>
+<robot name="xacro_properties" xmlns:xacro="http://ros.org/wiki/xacro">
+  <!-- Init colour -->
   <material name="black">
-    <color rgba="0.0 0.0 0.0 1.0"/>
+      <color rgba="0.0 0.0 0.0 1.0"/>
+  </material>
+  <material name="dark">
+    <color rgba="0.3 0.3 0.3 1.0"/>
+  </material>
+  <material name="light_black">
+    <color rgba="0.4 0.4 0.4 1.0"/>
   </material>
   <material name="blue">
@@ -12,5 +18,5 @@
   </material>
   <material name="grey">
-    <color rgba="0.2 0.2 0.2 1.0"/>
+    <color rgba="0.5 0.5 0.5 1.0"/>
   </material>
   <material name="orange">

File: src/rsk_bot/urdf/stereo_bot/stereo_bot.urdf.xacro (robot description, xacro)
@@ -5,5 +5,5 @@
   <xacro:property name="chassis_y" value="0.2"/>
   <xacro:property name="chassis_z" value="0.1"/>
-  <xacro:property name="chassis_mass" value="10"/>
+  <xacro:property name="chassis_mass" value="50"/>
   <xacro:property name="wheel_length" value="0.05"/>
   <xacro:property name="wheel_radius" value="0.1"/>
@@ -13,7 +13,7 @@
   <xacro:property name="cameraMass" value="0.1"/>
   <!-- Including File containing differential drive gazebo plugin -->
-  <xacro:include filename="$(find rsk_bot)/urdf/stereo_bot/plugin.gazebo" />
+  <xacro:include filename="$(find rsk_bot)/urdf/stereo_bot/stereo_bot.gazebo.xacro" />
   <!-- Including file containing materials information (colour) -->
-  <xacro:include filename="$(find rsk_bot)/urdf/stereo_bot/materials.xacro" />
+  <xacro:include filename="$(find rsk_bot)/urdf/common_properties.xacro" />
   <link name="dummy"> </link>
 <!-- ############################## Chassis  ####################################### -->
