Commit message: viso2 added

File: src/rsk_bot/urdf/mono_bot/mono_bot.gazebo.xacro (robot description, xacro)
@@ -36,13 +36,14 @@
       <material>Gazebo/Wood</material>
   </gazebo>
-  <!-- ################################# Gazebo Plugin for Stereo camera #############################-->
-   <gazebo reference="stereo_camera_link">
-    <sensor type="multicamera" name="stereo_camera">
+  <!-- ################################### Gazebo Plugin for Camera ###############################-->
+  <gazebo reference="camera_link">
+    <material>Gazebo/Green</material>
+    <sensor type="camera" name="camera">
       <update_rate>30.0</update_rate>
-      <camera name="left">
+      <camera name="head">
         <horizontal_fov>1.3962634</horizontal_fov>
         <image>
-          <width>800</width>
-          <height>800</height>
+          <width>400</width>
+          <height>400</height>
           <format>R8G8B8</format>
         </image>
@@ -51,42 +52,18 @@
           <far>300</far>
         </clip>
-        <noise>
-          <type>gaussian</type>
-          <mean>0.0</mean>
-          <stddev>0.007</stddev>
-        </noise>
       </camera>
-      <camera name="right">
-        <pose>0 -0.11 0 0 0 0</pose>
-        <horizontal_fov>1.3962634</horizontal_fov>
-        <image>
-          <width>800</width>
-          <height>800</height>
-          <format>R8G8B8</format>
-        </image>
-        <clip>
-          <near>0.02</near>
-          <far>300</far>
-        </clip>
-        <noise>
-          <type>gaussian</type>
-          <mean>0.0</mean>
-          <stddev>0.007</stddev>
-        </noise>
-      </camera>
-      <plugin name="stereo_camera_controller" filename="libgazebo_ros_multicamera.so">
-        <alwaysOn>              true                          </alwaysOn>
-        <updateRate>            0.0                           </updateRate>
-        <cameraName>            stereo                </cameraName>
-        <imageTopicName>        image_raw                     </imageTopicName>
-        <cameraInfoTopicName>   camera_info                   </cameraInfoTopicName>
-        <frameName>             stereo_camera_optical_link    </frameName>
-        <!--<rightFrameName>right_camera_optical_frame</rightFrameName>-->
-        <hackBaseline>          0.07                          </hackBaseline>
-        <distortionK1>          0.0                           </distortionK1>
-        <distortionK2>          0.0                           </distortionK2>
-        <distortionK3>          0.0                           </distortionK3>
-        <distortionT1>          0.0                           </distortionT1>
-        <distortionT2>          0.0                           </distortionT2>
+      <plugin name="camera_controller" filename="libgazebo_ros_camera.so">
+        <alwaysOn>              true                    </alwaysOn>
+        <updateRate>            10.0                    </updateRate>
+        <!--cameraName>            stereo_bot/left         </cameraName-->
+        <imageTopicName>        image             </imageTopicName>
+        <cameraInfoTopicName>   camera_info             </cameraInfoTopicName>
+        <frameName>             camera_optical_link             </frameName>
+        <hackBaseline>          0.07                    </hackBaseline>
+        <distortionK1>          0.0                     </distortionK1>
+        <distortionK2>          0.0                     </distortionK2>
+        <distortionK3>          0.0                     </distortionK3>
+        <distortionT1>          0.0                     </distortionT1>
+        <distortionT2>          0.0                     </distortionT2>
       </plugin>
     </sensor>

File: src/rsk_bot/urdf/mono_bot/mono_bot.urdf.xacro (robot description, xacro)
@@ -1,5 +1,5 @@
 <?xml version='1.0'?>
 <robot name="myrobot" xmlns:xacro="http://www.ros.org/wiki/xacro">
-  <xacro:include filename="$(find rsk_bot)/urdf/stereo_bot/stereo_bot.gazebo.xacro" />
+  <xacro:include filename="$(find rsk_bot)/urdf/mono_bot/mono_bot.gazebo.xacro" />
   <xacro:include filename="$(find rsk_bot)/urdf/common_properties.xacro" />
   <xacro:property name="chassis_x" value="0.4"/>
@@ -136,10 +136,10 @@
   </link>
   <!-- ######################################################################################################################## -->
-  <joint name="stereo_camera_joint" type="fixed">
-    <origin xyz="0.15 0.055 0.15" rpy="0 0 0"/>
+  <joint name="camera_joint" type="fixed">
+    <origin xyz="0.15 0 0.15" rpy="0 0 0"/>
     <parent link="base_link"/>
-    <child link="stereo_camera_link"/>
+    <child link="camera_link"/>
   </joint>
-  <link name="stereo_camera_link">
+  <link name="camera_link">
     <visual>
       <origin xyz="0 0 0" rpy="0 ${pi/2} 0"/>
@@ -162,10 +162,10 @@
   </link>
   <!-- ######################################################################################################################## -->
-   <joint name="stereo_camera_optical_joint" type="fixed">
+   <joint name="camera_optical_joint" type="fixed">
     <origin xyz="0 0 0" rpy="${-pi/2} 0 ${-pi/2}"/>
-    <parent link="stereo_camera_link"/>
-    <child link="stereo_camera_optical_link"/>
+    <parent link="camera_link"/>
+    <child link="camera_optical_link"/>
   </joint>
-  <link name="stereo_camera_optical_link"/>
+  <link name="camera_optical_link"/>
   <!-- ######################################################################################################################## -->
 </robot>
