Commit message: stereo_bot repaired

File: src/rsk_bot/urdf/stereo_bot/stereo_bot.gazebo.xacro (robot description, xacro)
@@ -4,31 +4,29 @@
   <gazebo>
     <plugin name="differential_drive_controller" filename="libgazebo_ros_diff_drive.so">
-    <!-- Here we need to provide different parameters of a differential drive Robot
-         that we made earlier -->
-      <legacyMode>          false                   </legacyMode>
-      <alwaysOn>            true                    </alwaysOn>
-      <updateRate>          20                      </updateRate>
-      <leftJoint>           left_wheel_hinge        </leftJoint>
-      <rightJoint>          right_wheel_hinge       </rightJoint>
-      <wheelSeparation>     0.4                     </wheelSeparation>
-      <wheelDiameter>       0.1                     </wheelDiameter>
-      <torque>              20                      </torque>
-      <commandTopic>        cmd_vel                 </commandTopic>
-      <odometryTopic>       odom                    </odometryTopic>
-      <odometryFrame>       odom                    </odometryFrame>
-      <robotBaseFrame>      base_link                 </robotBaseFrame>
-      <!-- I have used these to avoid warnings -->
-      <rosDebugLevel>na</rosDebugLevel>
-      <publishWheelTF> false </publishWheelTF>
-      <publishOdomTF> true </publishOdomTF>
-      <publishWheelJointState> false </publishWheelJointState>
-      <wheelAcceleration> 0 </wheelAcceleration>
-      <wheelTorque> 5 </wheelTorque>
-      <!-- <odometrySource> 1 </odometrySource> -->
-      <publishTf>1</publishTf>
+      <commandTopic>               cmd_vel              </commandTopic>
+      <odometryTopic>              odom                 </odometryTopic>
+      <odometryFrame>              odom                 </odometryFrame>
+      <odometrySource>             world                </odometrySource>
+      <publishOdomTF>              true                 </publishOdomTF>
+      <robotBaseFrame>             base_footprint       </robotBaseFrame>
+      <publishWheelTF>             false                </publishWheelTF>
+      <publishTf>                  true                 </publishTf>
+      <publishWheelJointState>     true                 </publishWheelJointState>
+      <legacyMode>                 false                </legacyMode>
+      <updateRate>                 30                   </updateRate>
+      <leftJoint>                  wheel_left_joint     </leftJoint>
+      <rightJoint>                 wheel_right_joint    </rightJoint>
+      <wheelSeparation>            0.4                  </wheelSeparation>
+      <wheelDiameter>              0.1                  </wheelDiameter>
+      <wheelAcceleration>          1                    </wheelAcceleration>
+      <wheelTorque>                20                   </wheelTorque>
+      <rosDebugLevel>              na                   </rosDebugLevel>
     </plugin>
   </gazebo>
-  <gazebo reference="chassis">
+  <gazebo reference="base_link">
       <material>Gazebo/WoodFloor</material>
+  </gazebo>
+  <gazebo reference="caster_link">
+      <material>Gazebo/Yellow</material>
   </gazebo>
   <gazebo reference="left_wheel">
@@ -58,8 +56,8 @@
         <alwaysOn>              true                    </alwaysOn>
         <updateRate>            10.0                    </updateRate>
-        <cameraName>            stereo_bot/left             </cameraName>
+        <cameraName>            sereo_bot/left             </cameraName>
         <imageTopicName>        image_raw               </imageTopicName>
         <cameraInfoTopicName>   camera_info             </cameraInfoTopicName>
-        <frameName>             point_cloud                  </frameName>
+        <frameName>             point_cloud             </frameName>
         <hackBaseline>          0.07                    </hackBaseline>
         <distortionK1>          0.0                     </distortionK1>
@@ -90,9 +88,9 @@
       <plugin name="camera_controller" filename="libgazebo_ros_camera.so">
         <alwaysOn>              true                    </alwaysOn>
-        <updateRate>            10.0                     </updateRate>
+        <updateRate>            10.0                    </updateRate>
         <cameraName>            stereo_bot/right            </cameraName>
         <imageTopicName>        image_raw               </imageTopicName>
         <cameraInfoTopicName>   camera_info             </cameraInfoTopicName>
-        <frameName>             point_cloud                  </frameName>
+        <frameName>             point_cloud             </frameName>
         <hackBaseline>          0.07                    </hackBaseline>
         <distortionK1>          0.0                     </distortionK1>

File: src/rsk_bot/urdf/stereo_bot/stereo_bot.urdf.xacro (robot description, xacro)
@@ -1,9 +1,10 @@
 <?xml version='1.0'?>
 <robot name="myrobot" xmlns:xacro="http://www.ros.org/wiki/xacro">
-<!-- xmlns:xacro="http://www.ros.org/wiki/xacro is also important dont know why -->
+  <xacro:include filename="$(find rsk_bot)/urdf/stereo_bot/stereo_bot.gazebo.xacro" />
+  <xacro:include filename="$(find rsk_bot)/urdf/common_properties.xacro" />
   <xacro:property name="chassis_x" value="0.4"/>
   <xacro:property name="chassis_y" value="0.2"/>
   <xacro:property name="chassis_z" value="0.1"/>
-  <xacro:property name="chassis_mass" value="50"/>
+  <xacro:property name="chassis_mass" value="10"/>
   <xacro:property name="wheel_length" value="0.05"/>
   <xacro:property name="wheel_radius" value="0.1"/>
@@ -12,14 +13,24 @@
   <xacro:property name="cameraLength" value="0.05"/>
   <xacro:property name="cameraMass" value="0.1"/>
-  <!-- Including File containing differential drive gazebo plugin -->
-  <xacro:include filename="$(find rsk_bot)/urdf/stereo_bot/stereo_bot.gazebo.xacro" />
-  <!-- Including file containing materials information (colour) -->
-  <xacro:include filename="$(find rsk_bot)/urdf/common_properties.xacro" />
-  <link name="dummy"> </link>
-<!-- ############################## Chassis  ####################################### -->
-  <!-- Chassis consists of two links : main_body and caster (spherical wheel) -->
-  <link name='chassis'>
-    <pose>0 0 0.1 0 0 0</pose>
-    <!-- Defining the inertia of whole chassis (main_body+caster) -->
+  <!-- ######################################################################################################################## -->
+  <link name="base_footprint"/>
+  <!-- ######################################################################################################################## -->
+  <joint name="base_joint" type="fixed">
+    <parent link="base_footprint"/>
+    <child link="base_link"/>
+    <origin xyz="0.0 0.0 0.010" rpy="0 0 0"/>
+  </joint>
+  <link name='base_link'>
+    <visual>
+      <origin xyz="0 0 0" rpy=" 0 0 0"/>
+      <geometry>
+        <box size="${chassis_x} ${chassis_y} ${chassis_z}"/>
+      </geometry>
+    </visual>
+    <collision>
+      <geometry>
+        <box size="${chassis_x} ${chassis_y} ${chassis_z}"/>
+      </geometry>
+    </collision>
     <inertial>
       <origin xyz="0 0 0.1" rpy=" 0 0 0"/>
@@ -29,27 +40,20 @@
         izz="${0.0833333 * chassis_mass * (chassis_x*chassis_x + chassis_y*chassis_y)}" />
     </inertial>
-    <!-- ~~~~~~~~~~~~~~~~~~~~~~~~~~~~~~~~~~~~~~~~~~~ -->
-    <!-- main_body's visual part and collision part is a cuboid  of size=".4 .2 .1" -->
-    <visual name='chassis_main_body_visual'>   <!--Visual name must have initials of link name in order to have color in gazebo-->
+  </link>
+  <!-- ######################################################################################################################## -->
+  <joint name="caster_joint" type="fixed">
+    <parent link="base_link"/>
+    <child link="caster_link"/>
+    <origin xyz="-0.15 0 -0.05" rpy="0 0 0"/>
+  </joint>
+  <link name='caster_link'>
+    <visual>
       <origin xyz="0 0 0" rpy=" 0 0 0"/>
-      <geometry>
-        <box size="${chassis_x} ${chassis_y} ${chassis_z}"/>
-      </geometry>
-    </visual>
-    <collision name='main_body_collision'>
-      <geometry>
-        <box size="${chassis_x} ${chassis_y} ${chassis_z}"/>
-      </geometry>
-    </collision>
-    <!-- ~~~~~~~~~~~~~~~~~~~~~~~~~~~~~~~~~~~~~~~~~~~ -->
-    <!-- caster wheel's visual part and collision part is a sphere  of radius="0.05" -->
-    <visual name='caster_visual'>
-      <origin xyz="-0.15 0 -0.05" rpy=" 0 0 0"/>
       <geometry>
         <sphere radius="0.05"/>
       </geometry>
     </visual>
-    <collision name='caster_collision'>
-      <origin xyz="-0.15 0 -0.05" rpy=" 0 0 0"/>
+    <collision>
+      <origin xyz="0 0 0" rpy=" 0 0 0"/>
       <geometry>
         <sphere radius="0.05"/>
@@ -67,7 +71,21 @@
     </collision>
   </link>
-  <!-- ############################## Left Wheel ####################################### -->
+  <!-- ######################################################################################################################## -->
+  <joint type="continuous" name="wheel_left_joint">
+    <origin xyz="0.1 0.15 0" rpy="0 0 0"/>
+    <child link="left_wheel"/>
+    <parent link="base_link"/>
+    <axis xyz="0 1 0" rpy="0 0 0"/>
+    <limit effort="100" velocity="100"/>
+    <joint_properties damping="0.0" friction="0.0"/>
+  </joint>
   <link name="left_wheel">
     <!--origin xyz="0.1 0.13 0.1" rpy="0 1.5707 1.5707"/-->
+    <visual name="left_wheel_visual">
+      <origin xyz="0 0 0" rpy="0 1.5707 1.5707"/>
+      <geometry>
+        <cylinder radius="${wheel_radius}" length="${wheel_length}"/>
+      </geometry>
+    </visual>
     <collision name="collision">
       <origin xyz="0 0 0" rpy="0 1.5707 1.5707"/>
@@ -76,10 +94,4 @@
       </geometry>
     </collision>
-    <visual name="left_wheel_visual">
-      <origin xyz="0 0 0" rpy="0 1.5707 1.5707"/>
-      <geometry>
-        <cylinder radius="${wheel_radius}" length="${wheel_length}"/>
-      </geometry>
-    </visual>
     <inertial>
       <origin xyz="0 0 0" rpy="0 1.5707 1.5707"/>
@@ -91,7 +103,21 @@
     </inertial>
   </link>
-  <!-- ############################## Right Wheel ####################################### -->
+  <!-- ######################################################################################################################## -->
+  <joint type="continuous" name="wheel_right_joint">
+    <origin xyz="0.1 -0.15 0" rpy="0 0 0"/>
+    <child link="right_wheel"/>
+    <parent link="base_link"/>
+    <axis xyz="0 1 0" rpy="0 0 0"/>
+    <limit effort="100" velocity="100"/>
+    <joint_properties damping="0.0" friction="0.0"/>
+  </joint>
   <link name="right_wheel">
     <!--origin xyz="0.1 -0.13 0.1" rpy="0 1.5707 1.5707"/-->
+    <visual name="right_wheel_visual">
+      <origin xyz="0 0 0" rpy="0 1.5707 1.5707"/>
+      <geometry>
+        <cylinder radius="${wheel_radius}" length="${wheel_length}"/>
+      </geometry>
+    </visual>
     <collision name="collision">
       <origin xyz="0 0 0" rpy="0 1.5707 1.5707"/>
@@ -100,10 +126,4 @@
       </geometry>
     </collision>
-    <visual name="right_wheel_visual">
-      <origin xyz="0 0 0" rpy="0 1.5707 1.5707"/>
-      <geometry>
-        <cylinder radius="${wheel_radius}" length="${wheel_length}"/>
-      </geometry>
-    </visual>
     <inertial>
       <origin xyz="0 0 0" rpy="0 1.5707 1.5707"/>
@@ -115,33 +135,12 @@
     </inertial>
   </link>
-  <joint name="dummy_joint" type="fixed">
-     <parent link="dummy"/>
-     <child link="chassis"/>
-   </joint>
-  <!-- ############################ Chassis to Left Wheel Joint ########################## -->
-  <joint type="continuous" name="left_wheel_hinge">
-    <origin xyz="0.1 0.15 0" rpy="0 0 0"/>
-    <child link="left_wheel"/>
-    <parent link="chassis"/>
-    <axis xyz="0 1 0" rpy="0 0 0"/>
-    <limit effort="100" velocity="100"/>
-    <joint_properties damping="0.0" friction="0.0"/>
+  <!-- ######################################################################################################################## -->
+  <joint name="left_camera_joint" type="fixed">
+    <axis xyz="0 1 0" />
+    <origin xyz="0.15 0.055 0.15" rpy="0 0 0"/>
+    <parent link="base_link"/>
+    <child link="left_camera"/>
   </joint>
-  <!-- ############################ Chassis to Right Wheel Joint ########################## -->
-  <joint type="continuous" name="right_wheel_hinge">
-    <origin xyz="0.1 -0.15 0" rpy="0 0 0"/>
-    <child link="right_wheel"/>
-    <parent link="chassis"/>
-    <axis xyz="0 1 0" rpy="0 0 0"/>
-    <limit effort="100" velocity="100"/>
-    <joint_properties damping="0.0" friction="0.0"/>
-  </joint>
-<!-- ############################## Left Camera  ####################################### -->
   <link name="left_camera">
-    <inertial>
-      <mass value="${cameraMass}" />
-      <origin xyz="0 0 0" rpy="0 0 0"/>
-      <inertia ixx="1e-6" ixy="0" ixz="0" iyy="1e-6" iyz="0" izz="1e-6" />
-    </inertial>
     <visual>
       <origin xyz="0 0 0" rpy="0 1.57075 0"/>
@@ -157,14 +156,4 @@
       </geometry>
     </collision>
-  </link>
-<!-- ############################## Chassis to Left Camera  ####################################### -->
-  <joint name="left_camera_joint" type="fixed">
-    <axis xyz="0 1 0" />
-    <origin xyz="0.15 0.055 0.15" rpy="0 0 0"/>
-    <parent link="chassis"/>
-    <child link="left_camera"/>
-  </joint>
-<!-- ############################## Right Camera  ####################################### -->
-  <link name="right_camera">
     <inertial>
       <mass value="${cameraMass}" />
@@ -172,4 +161,13 @@
       <inertia ixx="1e-6" ixy="0" ixz="0" iyy="1e-6" iyz="0" izz="1e-6" />
     </inertial>
+  </link>
+  <!-- ######################################################################################################################## -->
+  <joint name="right_camera_joint" type="fixed">
+    <axis xyz="0 1 0" />
+    <origin xyz="0.15 -0.055 0.15" rpy="0 0 0"/>
+    <parent link="base_link"/>
+    <child link="right_camera"/>
+  </joint>
+  <link name="right_camera">
     <visual>
       <origin xyz="0 0 0" rpy="0 1.57075 0"/>
@@ -185,39 +183,10 @@
       </geometry>
     </collision>
+    <inertial>
+      <mass value="${cameraMass}" />
+      <origin xyz="0 0 0" rpy="0 0 0"/>
+      <inertia ixx="1e-6" ixy="0" ixz="0" iyy="1e-6" iyz="0" izz="1e-6" />
+    </inertial>
   </link>
-<!-- ############################## Chassis to Right Camera  ####################################### -->
-  <joint name="right_camera_joint" type="fixed">
-    <axis xyz="0 1 0" />
-    <origin xyz="0.15 -0.055 0.15" rpy="0 0 0"/>
-    <parent link="chassis"/>
-    <child link="right_camera"/>
-  </joint>
-<!-- ############################## Point cloud (dummy link/frame) ####################################### -->
-  <link name="point_cloud">
-    <inertial>
-      <mass value="0" />
-      <origin xyz="0 0 0" rpy="0 0 0"/>
-      <inertia ixx="0" ixy="0" ixz="0" iyy="0" iyz="0" izz="0" />
-    </inertial>
-    <visual>
-      <origin xyz="0 0 0" rpy="0 0 0"/>
-      <geometry>
-        <sphere radius="0.01"/>
-      </geometry>
-      <material name="green"/>
-    </visual>
-    <collision>
-      <origin xyz="0 0 0" rpy="0 0 0"/>
-      <geometry>
-        <sphere radius="0.1"/>
-      </geometry>
-    </collision>
-  </link>
-<!-- ############################## Chassis to Point cloud  ####################################### -->
-  <joint name="point_cloud_joint" type="fixed">
-    <axis xyz="0 0 0" />
-    <origin xyz="0.15 0 0.05" rpy="4.712389 0 4.712389"/>
-    <parent link="chassis"/>
-    <child link="point_cloud"/>
-  </joint>
+  <!-- ######################################################################################################################## -->
 </robot>

File: src/rsk_bot/urdf/turtle_bot_burger/turtle_bot_burger.gazebo.xacro (robot description, xacro)
@@ -44,22 +44,22 @@
   <gazebo>
     <plugin name="turtlebot3_burger_controller" filename="libgazebo_ros_diff_drive.so">
-      <commandTopic>cmd_vel</commandTopic>
-      <odometryTopic>odom</odometryTopic>
-      <odometryFrame>odom</odometryFrame>
-      <odometrySource>world</odometrySource>
-      <publishOdomTF>true</publishOdomTF>
-      <robotBaseFrame>base_footprint</robotBaseFrame>
-      <publishWheelTF>false</publishWheelTF>
-      <publishTf>true</publishTf>
-      <publishWheelJointState>true</publishWheelJointState>
-      <legacyMode>false</legacyMode>
-      <updateRate>30</updateRate>
-      <leftJoint>wheel_left_joint</leftJoint>
-      <rightJoint>wheel_right_joint</rightJoint>
-      <wheelSeparation>0.160</wheelSeparation>
-      <wheelDiameter>0.066</wheelDiameter>
-      <wheelAcceleration>1</wheelAcceleration>
-      <wheelTorque>10</wheelTorque>
-      <rosDebugLevel>na</rosDebugLevel>
+      <commandTopic>               cmd_vel              </commandTopic>
+      <odometryTopic>              odom                 </odometryTopic>
+      <odometryFrame>              odom                 </odometryFrame>
+      <odometrySource>             world                </odometrySource>
+      <publishOdomTF>              true                 </publishOdomTF>
+      <robotBaseFrame>             base_footprint       </robotBaseFrame>
+      <publishWheelTF>             false                </publishWheelTF>
+      <publishTf>                  true                 </publishTf>
+      <publishWheelJointState>     true                 </publishWheelJointState>
+      <legacyMode>                 false                </legacyMode>
+      <updateRate>                 30                   </updateRate>
+      <leftJoint>                  wheel_left_joint     </leftJoint>
+      <rightJoint>                 wheel_right_joint    </rightJoint>
+      <wheelSeparation>            0.160                </wheelSeparation>
+      <wheelDiameter>              0.066                </wheelDiameter>
+      <wheelAcceleration>          1                    </wheelAcceleration>
+      <wheelTorque>                10                   </wheelTorque>
+      <rosDebugLevel>              na                   </rosDebugLevel>
     </plugin>
   </gazebo>

Commit message: stereo updated

File: src/rsk_bot/urdf/stereo_bot/stereo_bot.gazebo.xacro (robot description, xacro)
@@ -9,5 +9,5 @@
       <odometrySource>             world                </odometrySource>
       <publishOdomTF>              true                 </publishOdomTF>
-      <robotBaseFrame>             base_link       </robotBaseFrame>
+      <robotBaseFrame>             base_footprint       </robotBaseFrame>
       <publishWheelTF>             false                </publishWheelTF>
       <publishTf>                  true                 </publishTf>
@@ -78,5 +78,5 @@
         <alwaysOn>              true                          </alwaysOn>
         <updateRate>            0.0                           </updateRate>
-        <cameraName>            stereo                </cameraName>
+        <cameraName>            stereo_bot                </cameraName>
         <imageTopicName>        image_raw                     </imageTopicName>
         <cameraInfoTopicName>   camera_info                   </cameraInfoTopicName>

File: src/rsk_bot/urdf/stereo_bot/stereo_bot.urdf.xacro (robot description, xacro)
@@ -14,11 +14,11 @@
   <xacro:property name="cameraMass" value="0.1"/>
   <!-- ######################################################################################################################## -->
-  <!--link name="base_footprint"/-->
+  <link name="base_footprint"/>
   <!-- ######################################################################################################################## -->
-  <!--joint name="base_joint" type="fixed">
+  <joint name="base_joint" type="fixed">
     <parent link="base_footprint"/>
     <child link="base_link"/>
     <origin xyz="0.0 0.0 0.010" rpy="0 0 0"/>
-  </joint-->
+  </joint>
   <link name='base_link'>
     <visual>
